File: schem/fourth_year/fourth_year.sch (KiCad schematic (older format))
At the start: 0 parts

Commit message: filter test PCB mostly completed
Parts:
- added C?: 5.6pF, symbol C
- added C? (x8): 1nF, symbol C
- added C?: OPEN, symbol C
- added C?: 4.7pF, symbol C
- added C?: 8.2pF, symbol C
- added C?: 2pF, symbol C
- added C?: 0.47uF, symbol C
- added C?: 1.5nF, symbol C
- added C?: 33nF, symbol C
- added C? (x2): 26pF, symbol C
- added C?: 22pF, symbol C
- added C?: 1uF, symbol C
- added C?: C, symbol C
- added C? (x2): 1000pF, symbol C
- added K? (x2): CONN_3, symbol CONN_3
- added L? (x2): 270nH, symbol INDUCTOR
- added L?: 47nH, symbol INDUCTOR
- added L?: 18nH, symbol INDUCTOR
- added L?: 12nH, symbol INDUCTOR
- added L?: 19nH, symbol INDUCTOR
- added L?: 15nH, symbol INDUCTOR
- added L?: 68nH, symbol INDUCTOR
- added L?: 150nH, symbol INDUCTOR
- added L?: FERRITE BEAD, symbol INDUCTOR
- added P?: BNC, symbol BNC
- added P?: CONN_1, symbol CONN_1
- added P?: DC JACK, symbol BNC
- added R?: 600, symbol R
- added R?: 560, symbol R
- added R?: 15, symbol R
- added U?: MAX3543, symbol MAX3543
- added X?: CRYSTAL, symbol CRYSTAL
Connections:
- net labels added: 3V3, GND
- wire segments 0 -> 111

Commit message: Added ADC to model, updated schematic, created test data generator
Parts:
- added C?: 120uF, symbol C
- added C?: 150uF, symbol C
- added C?: 10uF, 1ohm ESR, symbol C
- added C? (x2): 3uF, symbol C
- added C? (x2): 10nF, symbol C
- added Q?: LT1086, symbol LT1086
- added Q?: UA78L05, symbol UA78L05
- added R? (x4): 500, symbol R
- added R? (x2): R, symbol R
- added U?: TPS7301, symbol TPS7301
- added U?: AD8138, symbol AD8138
- added U?: AD9235, symbol AD9235
Connections:
- net labels added: 3V, 5V
- wire segments 111 -> 174
Other:
- moved on the sheet: C?, L?, P?, R?, U?, X?

Commit message: Minor schem modifications, started final report
Parts:
- removed K? (x2): CONN_3, symbol CONN_3
- added C? (x2): 10uF, symbol C
- added C? (x4): .1uF, symbol C
- added R? (x2): 10K, symbol R
- added R? (x2): R, symbol R
- R?: value R -> 10K
- R?: value R -> 20K
Connections:
- wire segments 174 -> 209
Other:
- moved on the sheet: C?, L?, P?, Q?, R?, U?, X?

Commit message: Created fmc_lpc pad (see make_fmc_pads.py).  Broke up model src files.
Parts:
- added P?: SAW, symbol CONN_5
- added U?: FMC_LPC, symbol FMC_LPC
Connections:
- wire segments 209 -> 220
Other:
- moved on the sheet: C?, L?, P?, Q?, R?, U?, X?

Commit message: Some minor schematic work
Parts:
- removed P?: CONN_1, symbol CONN_1
- removed U?: FMC_LPC, symbol FMC_LPC
- added R?: OPEN / 360, ~, symbol R
- added U?: FMC_LPC, ~, symbol FMC_LPC
- C? (x2): value 1000pF -> 1nF
Connections:
- net labels added: SCL, SDA
- wire segments 220 -> 297
Other:
- note added: "2v5"

Commit message: Minor schematic updates
Parts:
- added C? (x2): .1uF, symbol C
- added L? (x3): OPEN, ~, symbol INDUCTOR
- added P3, P5: CONNECTOR, ~, symbol CONNECTOR
- added P? (x2): CONN_6, ~, symbol CONN_6
- added P?: BNC, symbol BNC
- added P? (x2): CONN_1, ~, symbol CONN_1
- added R15: R, ~, symbol R
- added R?: OPEN, ~, symbol R
- added T?: TRANSFO4, ~, symbol TRANSFO4
- C21: renamed from C?; value 22pF -> 18Pf
- C22: renamed from C?; value C -> 1nF
- C26: renamed from C?; value 120uF -> 150uF
- P1: renamed from P?; value BNC -> F Type
- gave numbers to parts that had none: 67
Connections:
- net labels removed: SCL, SDA
- wire segments 297 -> 310
Other:
- note added: "AA and Noise Supression\nFilter"
- note added: "Clapp Oscillator"
- note added: "Diplex Filter"
- note added: "Female Conn.\nTo BBB."
- note added: "For DC blocking"
- note added: "Function Generator\nInput"
- note added: "Matching Inductor"
- note added: "No idea what\nthis is for"
- note added: "PLL Charge Pump\n"
- note added: "R for Z matching"
- note added: "RF TAP?"
- moved on the sheet: C22, C29, C30, P4, U3

Commit message: Schematic complete.  Started work on pcb layout
Parts:
- removed C26, C29: 150uF, symbol C
- removed L? (x2): OPEN, ~, symbol INDUCTOR
- removed R4: 15, symbol R
- added C26, C29: 150uF, ~, symbol CP1
- added C37, C38: .1uF, 3.20mm x 1.60mm, symbol C
- added C39: 3pF, 2.00mm x 1.25mm, symbol C
- added C40, C41: 1uF, 3.20mmX1.60mm, symbol C
- added C42: 22uF, ~, symbol CP1
- added C43, C44: 45pF, 1.60mm x 0.80mm, symbol C
- added C45: 10uF, 2.00mm x 1.25mm, symbol C
- added C46: 82pF, 3.20mm x 1.60mm, symbol C
- added C49: 47uF, ~, symbol CP1
- added C50: 1uF, 3.20mm x 1.60mm, symbol C
- added C51: 100uF, ~, symbol CP1
- added C52: 3uF, ~, symbol C
- added D1: 1N5817, THROUGH HOLE, symbol DIODE
- added L12: FERRITE BEAD, 1.00mm x 0.50mm, symbol INDUCTOR
- added L18, L19: 112nH, 1.60mm x 0.80mm, symbol INDUCTOR
- added L21: 10uH, 3.20mm x 1.60mm, symbol INDUCTOR
- added L22: 22uH, 3.20mm x 1.60mm, symbol INDUCTOR
- added R16, R17: 120/SHORT, 3.20mm x 1.60mm, symbol R
- added U6, U7: 74VHC541FT, ~, symbol 74VHC541FT
- added U8: TPS6735, symbol TPS6735
- C1, C10, C11, C12, C13, C14, C15, C17, C18, C19, C2, C20, C22, C24, C25, C3, C31, C36, C4, C6, C7, C8: footprint (none) -> 2.00mm x 1.25mm
- C16: footprint (none) -> 1.25mm x 2.00mm WIDE
- C21: footprint (none) -> 1.00mm x 0.55mm
- C23: footprint (none) -> 2.30mm x 1.60mm
- C27, C28: footprint (none) -> 3.20mm x 2.50mm
- C30, C32, C33, C34, C35, C9, R10, R11, R12, R13, R14, R2, R7, R8, R9: footprint (none) -> 3.20mm x 1.60mm
- C47, C48: renamed from C?; footprint (none) -> 3.20mm x 1.60mm
- C5: value 5.6pF -> 3pF; footprint (none) -> 2.00mm x 1.25mm
- L1, L2, L3, L4, L5, L7, L8, L9: footprint (none) -> 1.60mm x 0.80mm
- L10: footprint (none) -> 1.00mm x 0.50mm
- L20: renamed from L?; footprint ~ -> 3.20mm x 1.60mm
- L6: footprint (none) -> 1.19mm x 0.64mm
- P1: footprint (none) -> F TYPE CONN
- P10: renamed from P?; footprint (none) -> BNC
- P2: footprint (none) -> SAW
- P3, P5: footprint ~ -> FEMALE CONN THROUGH HOLE
- P4: footprint (none) -> JACK
- P6, P7, P9: renamed from P?; footprint ~ -> THROUGH HOLE CONN
- R1: value 600 -> 50/OPEN; footprint (none) -> 3.20mm x 1.60mm
- R15: value R -> 50/OPEN; footprint ~ -> 3.20mm x 1.60mm
- R3: footprint ~ -> 2.00mm x 1.25mm
- R4: renamed from R?; value OPEN -> 100/OPEN; footprint ~ -> 3.20mm x 1.60mm
- R5, R6: value R -> 10K; footprint (none) -> 3.20mm x 1.60mm
- U3: value TPS7301 -> TPS7330QP
- U4: footprint (none) -> THROUGH HOLE CONN
- gave numbers to parts that had none: 2
Connections:
- net labels added: +2,5V, -5V, RF_IN
- wire segments 310 -> 433
Other:
- note added: "+"
- note added: "-"
- note added: "100 ohm"
- note added: "120 ohm"
- note added: "50 OHM LINES"
- note added: "75 OHM LINES"
- note added: "CLK"
- note added: "DRIVE WITH TRANSISTOR?"
- note added: "LINE DRIVERS"
- note added: "SEE SPICE MODEL\n& GENESYS"
- moved on the sheet: C1, C10, C11, C12, C13, C14, C15, C16, C17, C18, C19, C2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

Commit message: minor file updates
Parts:
- removed C10: 2pF, 2.00mm x 1.25mm, symbol C
- removed C6: 4.7pF, 2.00mm x 1.25mm, symbol C
- removed C8: 8.2pF, 2.00mm x 1.25mm, symbol C
- removed L7: 18nH, 1.60mm x 0.80mm, symbol INDUCTOR
- removed L8: 12nH, 1.60mm x 0.80mm, symbol INDUCTOR
Connections:
- wire segments 433 -> 426
Other:
- note added: "The high frequency\nside has been\neliminated"
Changed lines of the file:
@@
-$EndComp
-$Comp
-L INDUCTOR L8
-U 1 1 542CB867
-P 2400 6500
-F 0 "L8" V 2350 6500 40  0000 C CNN
-F 1 "12nH" V 2500 6500 40  0000 C CNN
-F 2 "1.60mm x 0.80mm" H 2400 6500 60  0001 C CNN
-F 3 "" H 2400 6500 60  0001 C CNN
-	1    2400 6500
-	-1   0    0    1
-$EndComp
-$Comp
-L GND #PWR051
-U 1 1 542CB85F
-P 2850 6950
-F 0 "#PWR051" H 2850 6950 30  0001 C CNN
-F 1 "GND" H 2850 6880 30  0001 C CNN
-F 2 "" H 2850 6950 60  0001 C CNN
-F 3 "" H 2850 6950 60  0001 C CNN
-	1    2850 6950
-	1    0    0    -1
-$EndComp
-$Comp
-L C C10
-U 1 1 542CB858
-P 2650 6850
-F 0 "C10" H 2700 6950 50  0000 L CNN
-F 1 "2pF" H 2700 6750 50  0000 L CNN
-F 2 "2.00mm x 1.25mm" H 2650 6850 60  0001 C CNN
-F 3 "" H 2650 6850 60  0001 C CNN
-	1    2650 6850
-	0    -1   -1   0
-$EndComp
-$Comp
-L C C8
-U 1 1 542CB82B
-P 2400 7050
-F 0 "C8" H 2450 7150 50  0000 L CNN
-F 1 "8.2pF" H 2450 6950 50  0000 L CNN
-F 2 "2.00mm x 1.25mm" H 2400 7050 60  0001 C CNN
-F 3 "" H 2400 7050 60  0001 C CNN
-	1    2400 7050
-	-1   0    0    1
-$EndComp
-$Comp
-L GND #PWR052
-U 1 1 542CB820
-P 2250 8050
-F 0 "#PWR052" H 2250 8050 30  0001 C CNN
-F 1 "GND" H 2250 7980 30  0001 C CNN
-F 2 "" H 2250 8050 60  0001 C CNN
-F 3 "" H 2250 8050 60  0001 C CNN
-	1    2250 8050
-	1    0    0    -1
-$EndComp
-$Comp
-L INDUCTOR L7
-U 1 1 542CB807
-P 2250 7600
-F 0 "L7" V 2200 7600 40  0000 C CNN
-F 1 "18nH" V 2350 7600 40  0000 C CNN
-F 2 "1.60mm x 0.80mm" H 2250 7600 60  0001 C CNN
-F 3 "" H 2250 7600 60  0001 C CNN
-	1    2250 7600
-	1    0    0    -1
-$EndComp
-$Comp
-L C C6
-U 1 1 542CB7FB
-P 2000 7300
-F 0 "C6" H 2050 7400 50  0000 L CNN
-F 1 "4.7pF" H 2050 7200 50  0000 L CNN
-F 2 "2.00mm x 1.25mm" H 2000 7300 60  0001 C CNN
-F 3 "" H 2000 7300 60  0001 C CNN
-	1    2000 7300
-	0    -1   -1   0
 $EndComp
 $Comp
@@
 $EndComp
 $Comp
-L GND #PWR053
+L GND #PWR051
 U 1 1 542CB715
 P 2050 6600
-F 0 "#PWR053" H 2050 6600 30  0001 C CNN
+F 0 "#PWR051" H 2050 6600 30  0001 C CNN
 F 1 "GND" H 2050 6530 30  0001 C CNN
 F 2 "" H 2050 6600 60  0001 C CNN
@@
 $EndComp
 $Comp
-L GND #PWR054
+L GND #PWR052
 U 1 1 542CB667
 P 800 7250
-F 0 "#PWR054" H 800 7250 30  0001 C CNN
+F 0 "#PWR052" H 800 7250 30  0001 C CNN
 F 1 "GND" H 800 7180 30  0001 C CNN
 F 2 "" H 800 7250 60  0001 C CNN
@@
 $EndComp
 $Comp
-L GND #PWR055
+L GND #PWR053
 U 1 1 542CB5CA
 P 1150 7750
-F 0 "#PWR055" H 1150 7750 30  0001 C CNN
+F 0 "#PWR053" H 1150 7750 30  0001 C CNN
 F 1 "GND" H 1150 7680 30  0001 C CNN
 F 2 "" H 1150 7750 60  0001 C CNN
@@
 $EndComp
 $Comp
-L GND #PWR056
+L GND #PWR054
 U 1 1 549DB423
 P 4800 7200
-F 0 "#PWR056" H 4800 7200 30  0001 C CNN
+F 0 "#PWR054" H 4800 7200 30  0001 C CNN
 F 1 "GND" H 4800 7130 30  0001 C CNN
 F 2 "" H 4800 7200 60  0000 C CNN
@@
 $EndComp
 $Comp
-L GND #PWR057
+L GND #PWR055
 U 1 1 54A2EC15
 P 6150 13050
-F 0 "#PWR057" H 6150 13050 30  0001 C CNN
+F 0 "#PWR055" H 6150 13050 30  0001 C CNN
 F 1 "GND" H 6150 12980 30  0001 C CNN
 F 2 "" H 6150 13050 60  0000 C CNN
@@
 $EndComp
 $Comp
-L GND #PWR058
+L GND #PWR056
 U 1 1 54A474CE
 P 15000 6950
-F 0 "#PWR058" H 15000 6950 30  0001 C CNN
+F 0 "#PWR056" H 15000 6950 30  0001 C CNN
 F 1 "GND" H 15000 6880 30  0001 C CNN
 F 2 "" H 15000 6950 60  0000 C CNN
@@
 $EndComp
 $Comp
-L GND #PWR059
+L GND #PWR057
 U 1 1 54A47755
 P 15550 6550
-F 0 "#PWR059" H 15550 6550 30  0001 C CNN
+F 0 "#PWR057" H 15550 6550 30  0001 C CNN
 F 1 "GND" H 15550 6480 30  0001 C CNN
 F 2 "" H 15550 6550 60  0000 C CNN
@@
 $EndComp
 $Comp
-L GND #PWR060
+L GND #PWR058
 U 1 1 54A48033
 P 15150 5500
-F 0 "#PWR060" H 15150 5500 30  0001 C CNN
+F 0 "#PWR058" H 15150 5500 30  0001 C CNN
 F 1 "GND" H 15150 5430 30  0001 C CNN
 F 2 "" H 15150 5500 60  0000 C CNN
@@
 $EndComp
 $Comp
-L GND #PWR061
+L GND #PWR059
 U 1 1 54A4818D
 P 14250 6400
-F 0 "#PWR061" H 14250 6400 30  0001 C CNN
+F 0 "#PWR059" H 14250 6400 30  0001 C CNN
 F 1 "GND" H 14250 6330 30  0001 C CNN
 F 2 "" H 14250 6400 60  0000 C CNN
@@
 $EndComp
 $Comp
-L +2,5V #PWR062
+L +2,5V #PWR060
 U 1 1 54A6D331
 P 6700 12350
-F 0 "#PWR062" H 6700 12300 20  0001 C CNN
+F 0 "#PWR060" H 6700 12300 20  0001 C CNN
 F 1 "+2,5V" H 6700 12450 30  0000 C CNN
 F 2 "" H 6700 12350 60  0000 C CNN
@@
 $EndComp
 $Comp
-L GND #PWR063
+L GND #PWR061
 U 1 1 54A6F84A
 P 11400 13250
-F 0 "#PWR063" H 11400 13250 30  0001 C CNN
+F 0 "#PWR061" H 11400 13250 30  0001 C CNN
 F 1 "GND" H 11400 13180 30  0001 C CNN
 F 2 "" H 11400 13250 60  0000 C CNN
@@
 $EndComp
 $Comp
-L GND #PWR064
+L GND #PWR062
 U 1 1 54A70377
 P 11400 11550
-F 0 "#PWR064" H 11400 11550 30  0001 C CNN
+F 0 "#PWR062" H 11400 11550 30  0001 C CNN
 F 1 "GND" H 11400 11480 30  0001 C CNN
 F 2 "" H 11400 11550 60  0000 C CNN
@@
 AA and Noise Supression\nFilter
 $Comp
-L GND #PWR065
+L GND #PWR063
 U 1 1 54416A75
 P 6100 5000
-F 0 "#PWR065" H 6100 5000 30  0001 C CNN
+F 0 "#PWR063" H 6100 5000 30  0001 C CNN
 F 1 "GND" H 6100 4930 30  0001 C CNN
 F 2 "" H 6100 5000 60  0001 C CNN
@@
 $EndComp
 $Comp
-L 5V #PWR066
+L 5V #PWR064
 U 1 1 54A909B2
 P 18200 3100
-F 0 "#PWR066" H 18200 3200 40  0001 C CNN
+F 0 "#PWR064" H 18200 3200 40  0001 C CNN
 F 1 "5V" H 18200 3275 40  0000 C CNN
 F 2 "~" H 18200 3100 60  0000 C CNN
@@
 $EndComp
 $Comp
-L GND #PWR067
+L GND #PWR065
 U 1 1 54A90D4B
 P 18800 3550
-F 0 "#PWR067" H 18800 3550 30  0001 C CNN
+F 0 "#PWR065" H 18800 3550 30  0001 C CNN
 F 1 "GND" H 18800 3480 30  0001 C CNN
 F 2 "" H 18800 3550 60  0000 C CNN
@@
 $EndComp
 $Comp
-L 5V #PWR068
+L 5V #PWR066
 U 1 1 54A90F27
 P 16650 3300
-F 0 "#PWR068" H 16650 3400 40  0001 C CNN
+F 0 "#PWR066" H 16650 3400 40  0001 C CNN
 F 1 "5V" H 16650 3475 40  0000 C CNN
 F 2 "~" H 16650 3300 60  0000 C CNN
@@
 $EndComp
 $Comp
-L GND #PWR069
+L GND #PWR067
 U 1 1 54A912E5
 P 16150 4200
-F 0 "#PWR069" H 16150 4200 30  0001 C CNN
+F 0 "#PWR067" H 16150 4200 30  0001 C CNN
 F 1 "GND" H 16150 4130 30  0001 C CNN
 F 2 "" H 16150 4200 60  0000 C CNN
@@
 $EndComp
 $Comp
-L GND #PWR070
+L GND #PWR068
 U 1 1 54A9169A
 P 16600 4650
-F 0 "#PWR070" H 16600 4650 30  0001 C CNN
+F 0 "#PWR068" H 16600 4650 30  0001 C CNN
 F 1 "GND" H 16600 4580 30  0001 C CNN
 F 2 "" H 16600 4650 60  0000 C CNN
@@
 $EndComp
 $Comp
-L GND #PWR071
+L GND #PWR069
 U 1 1 54A91878
 P 18200 3950
-F 0 "#PWR071" H 18200 3950 30  0001 C CNN
+F 0 "#PWR069" H 18200 3950 30  0001 C CNN
 F 1 "GND" H 18200 3880 30  0001 C CNN
 F 2 "" H 18200 3950 60  0000 C CNN
@@
 $EndComp
 $Comp
-L GND #PWR072
+L GND #PWR070
 U 1 1 54A91A68
 P 18700 4400
-F 0 "#PWR072" H 18700 4400 30  0001 C CNN
+F 0 "#PWR070" H 18700 4400 30  0001 C CNN
 F 1 "GND" H 18700 4330 30  0001 C CNN
 F 2 "" H 18700 4400 60  0000 C CNN
@@
 $EndComp
 $Comp
-L GND #PWR073
+L GND #PWR071
 U 1 1 54A92BBF
 P 19600 4250
-F 0 "#PWR073" H 19600 4250 30  0001 C CNN
+F 0 "#PWR071" H 19600 4250 30  0001 C CNN
 F 1 "GND" H 19600 4180 30  0001 C CNN
 F 2 "" H 19600 4250 60  0000 C CNN
@@
 $EndComp
 $Comp
-L GND #PWR074
+L GND #PWR072
 U 1 1 54A93378
 P 20350 4250
-F 0 "#PWR074" H 20350 4250 30  0001 C CNN
+F 0 "#PWR072" H 20350 4250 30  0001 C CNN
 F 1 "GND" H 20350 4180 30  0001 C CNN
 F 2 "" H 20350 4250 60  0000 C CNN
@@
 $EndComp
 $Comp
-L -5V #PWR075
+L -5V #PWR073
 U 1 1 54A93941
 P 20500 3550
-F 0 "#PWR075" H 20500 3690 20  0001 C CNN
+F 0 "#PWR073" H 20500 3690 20  0001 C CNN
 F 1 "-5V" H 20500 3660 30  0000 C CNN
 F 2 "" H 20500 3550 60  0000 C CNN
@@
 $EndComp
 $Comp
-L GND #PWR076
+L GND #PWR074
 U 1 1 54A93982
 P 7800 4550
-F 0 "#PWR076" H 7800 4550 30  0001 C CNN
+F 0 "#PWR074" H 7800 4550 30  0001 C CNN
 F 1 "GND" H 7800 4480 30  0001 C CNN
 F 2 "" H 7800 4550 60  0000 C CNN
@@
 $EndComp
 $Comp
-L GND #PWR077
+L GND #PWR075
 U 1 1 54A9415D
 P 7900 7000
-F 0 "#PWR077" H 7900 7000 30  0001 C CNN
+F 0 "#PWR075" H 7900 7000 30  0001 C CNN
 F 1 "GND" H 7900 6930 30  0001 C CNN
 F 2 "" H 7900 7000 60  0000 C CNN
@@
 $EndComp
 $Comp
-L -5V #PWR078
+L -5V #PWR076
 U 1 1 54A9416C
 P 7900 6400
-F 0 "#PWR078" H 7900 6540 20  0001 C CNN
+F 0 "#PWR076" H 7900 6540 20  0001 C CNN
 F 1 "-5V" H 7900 6510 30  0000 C CNN
 F 2 "" H 7900 6400 60  0000 C CNN
@@
 $EndComp
 $Comp
-L GND #PWR079
+L GND #PWR077
 U 1 1 54A9FA00
 P 12350 11800
-F 0 "#PWR079" H 12350 11800 30  0001 C CNN
+F 0 "#PWR077" H 12350 11800 30  0001 C CNN
 F 1 "GND" H 12350 11730 30  0001 C CNN
 F 2 "" H 12350 11800 60  0000 C CNN
@@
 $EndComp
 $Comp
-L GND #PWR080
+L GND #PWR078
 U 1 1 54AA03B4
 P 12500 10000
-F 0 "#PWR080" H 12500 10000 30  0001 C CNN
+F 0 "#PWR078" H 12500 10000 30  0001 C CNN
 F 1 "GND" H 12500 9930 30  0001 C CNN
 F 2 "" H 12500 10000 60  0000 C CNN
@@
 $EndComp
 $Comp
-L GND #PWR081
+L GND #PWR079
 U 1 1 54AAE2EF
 P 18850 1900
-F 0 "#PWR081" H 18850 1900 30  0001 C CNN
+F 0 "#PWR079" H 18850 1900 30  0001 C CNN
 F 1 "GND" H 18850 1830 30  0001 C CNN
 F 2 "" H 18850 1900 60  0000 C CNN
@@
 Wire Wire Line
 	2550 5700 1100 5700
-Wire Wire Line
-	1800 7150 1800 7300
-Wire Wire Line
-	2850 6850 2850 6950
-Wire Wire Line
-	2200 7300 2400 7300
-Wire Wire Line
-	2400 7300 2400 7250
-Wire Wire Line
-	2250 7900 2250 8050
 Connection ~ 1550 7150
-Wire Wire Line
-	1400 7150 1800 7150
 Connection ~ 1550 6450
 Wire Wire Line
@@
 Wire Wire Line
 	1250 7050 1550 7050
-Connection ~ 2250 7300
-Wire Wire Line
-	2450 6850 2400 6850
-Wire Wire Line
-	2400 6850 2400 6800
-Wire Wire Line
-	2400 6200 3200 6200
 Wire Wire Line
 	1550 7450 1350 7450
@@
 Text Label 1550 7350 0    60   ~ 0
 RF_IN
+Wire Wire Line
+	1400 7150 1550 7150
+Text Notes 2100 7150 0    60   ~ 0
+The high frequency\nside has been\neliminated
+$Comp
+L GND #PWR080
+U 1 1 54AB0E46
+P 3200 6350
+F 0 "#PWR080" H 3200 6350 30  0001 C CNN
+F 1 "GND" H 3200 6280 30  0001 C CNN
+F 2 "" H 3200 6350 60  0000 C CNN
+F 3 "" H 3200 6350 60  0000 C CNN
+	1    3200 6350
+	1    0    0    -1
+$EndComp
+Wire Wire Line
+	3200 6350 3200 6200
 $EndSCHEMATC
